File: LIEF-P0/lief-p0r1.brd (EAGLE design)
At the start: 45 x 45 mm, 14 parts, among them U1 MPL3115A2LGA8, U2 L3G4200D, U3 HMC6343A

Commit message: Revision 3 of the LIEF hardware design.
Parts:
- added C10: 4.7uF, SparkFun-Capacitors:0805-CAP
- added C11: 0.22uF, SparkFun-Capacitors:0805-CAP
- added C7: 0.1uF, SparkFun-Capacitors:0603-CAP
- added C9: 4.7uF, SparkFun-Capacitors:0603-CAP
- added U$1: FT200XD, Synapseware:DFN-10
- added U4: (no value), bitfab:HMC5983-LPCC16
- JP1: device SparkFun-Connectors:1X10_LOCK -> pinhead:1X04
- JP2: device SparkFun-Connectors:1X04_LOCK -> pinhead:1X07
- U3: value HMC6343A -> MMA8452Q; device SparkFun-Sensors:LCC36 -> SparkFun-Sensors:QFN-16_0.5MM
- moved JP2 62.7 mm to (-3.77, -18.0)
- moved JP1 47.2 mm to (-7.58, -12.4), turned to 0 degrees
- moved U3 32.7 mm to (-1.78, 2.88), turned to 0 degrees
Connections:
- removed net N$1: JP1.10, U1.5
- removed net N$2: U3.22, U3.35
- removed net N$3: JP1.9, U1.6
- removed net N$4: JP1.7, U2.7
- new net ACCINT1: JP2.5
- new net ACCINT2: JP2.6
- new net ALTINT1: JP2.3
- new net ALTINT2: JP2.4
- new net COMPINT1: JP2.7
- new net GYROINT1: JP2.1
- new net GYROINT2: JP2.2
- new net N$10: C11.2, U4.SETP
- new net N$12: C10.1, U4.C1
- new net N$19: U4.DRDY
- new net N$9: C7.1, U3.2
- net 3V3: now also JP1.1, U3.1, U3.14, U4.I2C/SPI, U4.SPI_CS/S1, U4.SPI_SDO, U4.VDD, U4.VDDIO; no longer JP2.1, U3.11, U3.21, U3.3
- net GND: now also C10.2, C7.2, JP1.2, JP1.3, U3.10, U3.12, U3.5, U3.7, U4.GND, U4.SOC; no longer JP2.2, U3.25, U3.29
- net N$5: now also C11.1, U4.SETC; no longer JP1.8, U2.6
- net SCL: now also JP1.4, U3.4, U4.SCL/SPI_SCK; no longer JP2.4, U3.32
- net SDA: now also U3.6, U4.SDA/SPI_SDI; no longer JP2.3, U3.36
Routing:
- net N$2: track 58.2 -> 0.00 mm, vias 2 -> 0
- net N$4: track 26.9 -> 0.00 mm, vias 1 -> 0
- net N$5: track 22.7 -> 0.00 mm, vias 1 -> 0
- net GND: track 132.0 -> 114.0 mm
- net N$3: track 13.5 -> 0.00 mm
- net SCL: track 64.9 -> 55.2 mm
- net 3V3: track 141.5 -> 131.8 mm
- net N$1: track 8.92 -> 0.00 mm
- net SDA: track 86.6 -> 84.5 mm
