File: LIEF-P0/lief-p0r2.brd (EAGLE design)
At the start: 45 x 45 mm, 14 parts, among them U1 MPL3115A2LGA8, U2 L3G4200D, U3 HMC6343A

Commit message: Revision 3 of the LIEF hardware design.
Parts:
- removed R1, R2: 10K, resistor:M0805
- added C10: 4.7uF, SparkFun-Capacitors:0805-CAP
- added C11: 0.22uF, SparkFun-Capacitors:0805-CAP
- added C12, C8: 0.1uF, MySMD:CAP0805-NP
- added C7: 0.1uF, SparkFun-Capacitors:0603-CAP
- added C9: 4.7uF, SparkFun-Capacitors:0603-CAP
- added D1: MBR0520, MySMD:SOD-123
- added J3: USB-MINI-B%C, MyCON2:USB-MINI-B_2
- added LED1: RED_RX, MySMD:LED0805
- added LED2: GREEN_TX, MySMD:LED0805
- added LED4: GREEN_PWR, MySMD:LED0805
- added RP1, RP2: 330, MySMD:RES4NT
- added U4: (no value), bitfab:HMC5983-LPCC16
- added U5: FT232RL, MySMD2:SSOP28
- added U6: UA78M05, MySMD:SOT223
- added U7: AT90CAN-GENERIC-A, at90can32_64_128:TQFP64
- JP1: device SparkFun-Connectors:1X10_LOCK -> pinhead:1X04
- JP2: device SparkFun-Connectors:1X04_LOCK -> pinhead:1X07
- R3: device resistor:R0805 -> resistor:0204V
- U3: value HMC6343A -> MMA8452Q; device SparkFun-Sensors:LCC36 -> SparkFun-Sensors:QFN-16_0.5MM
- moved JP2 62.7 mm to (-3.77, -18.0)
- moved JP1 47.2 mm to (-7.58, -12.4), turned to 0 degrees
- moved U3 32.7 mm to (-1.78, 2.88), turned to 0 degrees
Connections:
- new net +5V: D1.1, LED1.2, LED2.2, RP1.2, U5.20, U5.4, U6.3
- new net ACCINT1: JP2.5, U3.11
- new net ACCINT2: JP2.6, U3.9
- new net ALTINT1: JP2.3, U1.6
- new net ALTINT2: JP2.4, U1.5
- new net AVCC: U7.64
- new net COM: C12.2
- new net COMPINT1: JP2.7, U4.DRDY
- new net GYROINT1: JP2.1, U2.7
- new net GYROINT2: JP2.2, U2.6
- new net N$10: C11.2, U4.SETP
- new net N$11: RP2.3, U5.23
- new net N$12: C10.1, U4.C1
- new net N$13: RP2.4, U5.22
- new net N$14: U5.11
- new net N$15: U5.6
- new net N$16: U5.8
- new net N$17: U5.9
- new net N$18: U5.10
- new net N$19: U5.28
- new net N$20: U5.27
- new net N$21: U5.24
- new net N$22: U5.13
- new net N$23: U5.14
- new net N$24: U5.12
- new net N$25: U5.19
- new net N$26: U5.26
- new net N$27: U5.3
- new net N$28: LED1.1, RP2.6
- new net N$29: LED2.1, RP2.5
- new net N$9: C7.1, U3.2
- new net RESET: C8.1
- new net RX: U5.1
- new net TX: U5.5
- new net VCC: U7.21, U7.52
- new net VIN: JP1.1, U6.1
- new net VUSB: D1.2, J3.5
- net 3V3: now also C12.1, U3.1, U3.14, U4.I2C/SPI, U4.SPI_CS/S1, U4.SPI_SDO, U4.VDD, U4.VDDIO, U5.17; no longer JP2.1, R1.2, R2.2, U3.11, U3.21, U3.3
- net GND: now also C10.2, C7.2, J3.1, J3.6, J3.7, J3.8, J3.9, JP1.2, JP1.3, LED4.1, U3.10, U3.12, U3.5, U3.7, U4.GND, U4.SOC, U5.18, U5.21, U5.25, U5.7, U6.2, U6.4, U7.22, U7.53, U7.63; no longer JP2.2, U3.25, U3.29
- net N$1: now also LED4.2, RP1.7; no longer JP1.10, U1.5
- net N$2: now also J3.3, U5.15; no longer U3.22, U3.35
- net N$3: now also J3.4, U5.16; no longer JP1.9, U1.6
- net N$4: now also C8.2, U5.2; no longer JP1.7, U2.7
- net N$5: now also C11.1, U4.SETC; no longer JP1.8, U2.6
- net SCL: now also JP1.4, U3.4, U4.SCL/SPI_SCK; no longer JP2.4, R2.1, U3.32
- net SDA: now also U3.6, U4.SDA/SPI_SDI; no longer JP2.3, R1.1, U3.36
Routing:
- net 3V3: track 141.9 -> 81.2 mm
- net N$2: track 58.2 -> 0.00 mm, vias 2 -> 0
- net SCL: track 65.2 -> 18.2 mm
- net N$4: track 26.9 -> 0.00 mm, vias 1 -> 0
- net N$5: track 22.7 -> 0.00 mm, vias 1 -> 0
- net GND: track 133.1 -> 114.0 mm
- net SDA: track 86.9 -> 69.8 mm
- net N$3: track 13.5 -> 0.00 mm
- net N$14: track 11.9 -> 0.00 mm
- net N$1: track 8.92 -> 0.00 mm
- net N$15: track 8.41 -> 0.00 mm
- net N$13: track 2.12 -> 0.00 mm
- removed copper zone on layer 16, net N$10
- removed copper zone on layer 16, net N$11
- removed copper zone on layer 16, net N$12
