File: LIEF-P0/lief-p0r2.sch (EAGLE design)
At the start: 14 parts, among them U1 MPL3115A2LGA8, U2 L3G4200D, U3 HMC6343A

Commit message: Revision 3 of the LIEF hardware design.
Parts:
- removed R1, R2: 10K, resistor:R-US_M0805
- added C10: 4.7uF, SparkFun-Capacitors:1.0UF-25V-+80/-20(0805)"
- added C11: 0.22uF, SparkFun-Capacitors:1.0UF-25V-+80/-20(0805)"
- added C12, C8: 0.1uF, MySMD:CAP0805-NP
- added C7: 0.1uF, SparkFun-Capacitors:0.1UF-100V-10%(0603)
- added C9: 4.7uF, SparkFun-Capacitors:0.1UF-100V-10%(0603)
- added D1: MBR0520, MySMD:MBR0520
- added J3: USB-MINI-B%C, MyCON2:USB-MINI-B%C
- added LED1: RED_RX, MySMD:LED0805
- added LED2: GREEN_TX, MySMD:LED0805
- added LED4: GREEN_PWR, MySMD:LED0805
- added RP1, RP2: 330, MySMD:RES4NT
- added U4: (no value), bitfab:HMC5983
- added U5: FT232RL, MySMD2:FT232RL
- added U6: UA78M05, MySMD:UA78M05
- added U7: AT90CAN-GENERIC-A, at90can32_64_128:AT90CAN-GENERIC-A
- JP1: device SparkFun-Connectors:M10LOCK -> pinhead:PINHD-1X4
- JP2: device SparkFun-Connectors:M04LOCK -> pinhead:PINHD-1X7
- R3: device resistor:R-US_R0805 -> resistor:R-US_0204/2V
- U3: value HMC6343A -> MMA8452Q; device SparkFun-Sensors:HMC6343A -> SparkFun-Sensors:MMA8452Q
Connections:
- new net +5V: D1.CA, LED1.AN, LED2.AN, RP1B.1, U5.VCC, U5.VCCIO, U6.OUT
- new net ACCINT1: JP2.5, U3.INT1
- new net ACCINT2: JP2.6, U3.INT2
- new net ALTINT1: JP2.3, U1.INT1
- new net ALTINT2: JP2.4, U1.INT2
- new net COM: C12.2
- new net COMPINT1: JP2.7, U4.DRDY
- new net GYROINT1: JP2.1, U2.INT1
- new net GYROINT2: JP2.2, U2.INT2
- new net N$10: C11.2, U4.SETP
- new net N$11: RP2C.1, U5.CBUS0
- new net N$12: C10.1, U4.C1
- new net N$13: RP2D.1, U5.CBUS1
- new net N$14: U5.CTS#
- new net N$15: U5.RI#
- new net N$16: U5.NC1
- new net N$17: U5.DSR#
- new net N$18: U5.DCD#
- new net N$19: U5.OSCO
- new net N$20: U5.OSCI
- new net N$21: U5.NC2
- new net N$22: U5.CBUS2
- new net N$23: U5.CBUS3
- new net N$24: U5.CBUS4
- new net N$25: U5.RESET#
- new net N$26: U5.TEST
- new net N$27: U5.RTS#
- new net N$28: LED1.CA, RP2C.2
- new net N$29: LED2.CA, RP2D.2
- new net N$9: C7.1, U3.BYP
- new net RESET: C8.1
- new net RX: U5.TXD
- new net TX: U5.RXD
- new net VIN: JP1.1, U6.IN
- new net VUSB: D1.AN, J3.VBUS
- net 3V3: now also C12.1, U3.VDD, U3.VDDIO, U4.I2C/SPI, U4.SPI_CS, U4.SPI_SDO, U4.VDD, U4.VDDIO, U5.3V3OUT; no longer JP2.1, R1.2, R2.2, U3.VDD@11, U3.VDD@21, U3.VDD@3
- net GND: now also C10.2, C7.2, J3.GND, J3.SH1, J3.SH2, J3.SH3, J3.SH4, JP1.2, JP1.3, LED4.CA, U3.GND@0, U3.GND@1, U3.GND@2, U3.SA0, U4.GND, U4.SOC, U5.AGND, U5.GND1, U5.GND2, U5.GND3, U6.GND1, U6.GND2; no longer JP2.2, U3.GND@25, U3.GND@29
- net N$1: now also LED4.AN, RP1B.2; no longer JP1.10, U1.INT2
- net N$2: now also J3.D+, U5.USBDP; no longer U3.CS, U3.CSC
- net N$3: now also J3.D-, U5.USBDM; no longer JP1.9, U1.INT1
- net N$4: now also C8.2, U5.DTR#; no longer JP1.7, U2.INT1
- net N$5: now also C11.1, U4.SETC; no longer JP1.8, U2.INT2
- net SCL: now also JP1.4, U4.SCL/SCK; no longer JP2.4, R2.1
- net SDA: now also U4.SDA/SDI; no longer JP2.3, R1.1
Other:
- note added: "1 mA"
- note added: "2 mA"
- note added: "3.0"
- note added: "5V Regulator"
- note added: "5V USB/VIN "Selector""
- note added: "7 mA"
- note added: "Accelerometer"
- note added: "Altimeter & Thermometer"
- note added: "BITFAB TECHNOLOGIES LLC"
- note added: "Board-to-Board Interface Header 1"
- note added: "Compass"
- note added: "Gyroscope"
- note added: "I2C address: 0x1D (7bit)"
- note added: "I2C address: 0x1E (7bit)"
- note added: "I2C address: 0x60 (7bit) 0xC1 (8bit read) 0xC0 (8bit write)"
- note added: "I2C address: 0x68 (7bit)"
- note added: "Interrupt Header 1"
- note added: "Power Filter"
- note added: "Todo ==== * connect the FTDI FT200XD * reduce power filter (see arduino schem) * add CBUS (ethernet) connector * check packages of all parts * enhance FT200XD symbol * coalesce all parts into bitfab.lbr"
- note added: "USB to Serial UART (RS232/422/485) & 3V3 Regulator"
- note added: "VCC := 5V (TTL) VDD := 3.3V (MOS)"
- note removed: "I2C address: 0x68"
- moved on the sheet: C1, C2, C3, C4, C5, C6, R3, U1, U2
